Commit message: updated Tuesday

File: src/agv_description/urdf/agv_description.gazebo.xacro (robot description, xacro)
@@ -5,8 +5,8 @@
             <legacyMode>false</legacyMode>
             <alwaysOn>true</alwaysOn>
-            <publishWheelTF>true</publishWheelTF>
-            <publishTf>1</publishTf>
+            <publishWheelTF>false</publishWheelTF>
+            <publishTf>true</publishTf>
             <publishWheelJointState>true</publishWheelJointState>
-            <updateRate>1</updateRate>
+            <updateRate>30</updateRate>
             <leftJoint>right_wheel_joint</leftJoint>
             <rightJoint>left_wheel_joint</rightJoint>
@@ -19,5 +19,5 @@
             <odometryTopic>odom</odometryTopic>
             <odometryFrame>odom</odometryFrame>
-	    <odometrySource></odometrySource>
+	    <odometrySource>world</odometrySource>
 	    <publishOdomTF>True</publishOdomTF>
             <robotBaseFrame>base_link</robotBaseFrame>

File: src/agv_description/urdf/agv_description.xacro (robot description, xacro)
@@ -20,5 +20,10 @@
         <inertia  ixx="${m*(3*r*r+h*h)/12}" ixy = "0" ixz = "0" iyy="${m*(3*r*r+h*h)/12}" iyz = "0" izz="${m*r*r/2}" />
     </xacro:macro>
-    <link name="odom"/>
+   	<!--<link name="odom"/>
+	<joint name="odom_foot" type="fixed">
+		<parent link="odom"/>
+		<child link="base_footprint"/>
+	</joint>-->
+	<link name="base_footprint"/>
     <link name="base_link">
 		<inertial>
@@ -41,12 +46,7 @@
         </collision>
     </link>
-    <!--<joint name="base_joint" type="fixed">
-    	<parent link="world"/>
-    	<child link="base_footprint"/>
-    	<origin xyz="0 0 0" rpy="0 0 0"/>
-    </joint>-->
     <joint name="base_link_joint" type="fixed">
-    	<origin xyz="0 0 0.05" rpy="0 0 0" />
-        <parent link="odom"/>
+    	<origin xyz="0 0 0.010" rpy="0 0 0" />
+        <parent link="base_footprint"/>
         <child link="base_link"/>
     </joint>
